Commit message: URDF提交

File: resources/robots/lmf1/model.urdf (robot description, URDF)
Before this commit: robot quadrotor, 5 links, 4 joints
Links:
- added link back_left_payload, mass 1.0; collision cylinder length=0.05 radius=0.07; visual cylinder length=0.05 radius=0.07
- added link back_left_support_drone, mass 1.0; collision box size=0.5 0.5 0.5; visual box size=0.4 0.4 0.025
- added link back_right_payload, mass 1.0; collision cylinder length=0.05 radius=0.07; visual cylinder length=0.05 radius=0.07
- added link back_right_support_drone, mass 1.0; collision box size=0.5 0.5 0.5; visual box size=0.4 0.4 0.025
- added link front_left_payload, mass 1.0; collision cylinder length=0.05 radius=0.07; visual cylinder length=0.05 radius=0.07
- added link front_left_support_drone, mass 1.0; collision box size=0.5 0.5 0.5; visual box size=0.4 0.4 0.025
- added link front_right_payload, mass 1.0; collision cylinder length=0.05 radius=0.07; visual cylinder length=0.05 radius=0.07
- added link front_right_support_drone, mass 1.0; collision box size=0.5 0.5 0.5; visual box size=0.4 0.4 0.025
- link base_link: mass 1.195 -> 8.0
Joints:
- added joint back_left_support_drone_to_payload: type fixed, parent back_left_support_drone, child back_left_payload, origin xyz=0 0 -0.15
- added joint back_right_support_drone_to_payload: type fixed, parent back_right_support_drone, child back_right_payload, origin xyz=0 0 -0.15
- added joint base_link_to_back_left_support_drone: type fixed, parent base_link, child back_left_support_drone, origin xyz=-0.282842 0.282842 -0.4
- added joint base_link_to_back_right_support_drone: type fixed, parent base_link, child back_right_support_drone, origin xyz=-0.282842 -0.282842 -0.4
- added joint base_link_to_front_left_support_drone: type fixed, parent base_link, child front_left_support_drone, origin xyz=0.282842 0.282842 -0.4
- added joint base_link_to_front_right_support_drone: type fixed, parent base_link, child front_right_support_drone, origin xyz=0.282842 -0.282842 -0.4
- added joint front_left_support_drone_to_payload: type fixed, parent front_left_support_drone, child front_left_payload, origin xyz=0 0 -0.15
- added joint front_right_support_drone_to_payload: type fixed, parent front_right_support_drone, child front_right_payload, origin xyz=0 0 -0.15

Commit message: 调整lmf2_controller_config的参数

File: resources/robots/lmf1/model.urdf (robot description, URDF)
Before this commit: robot quadrotor, 13 links, 12 joints
Links:
- removed link back_left_payload
- removed link back_left_support_drone
- removed link back_right_payload
- removed link back_right_support_drone
- removed link front_left_payload
- removed link front_left_support_drone
- removed link front_right_payload
- removed link front_right_support_drone
- link base_link: mass 8.0 -> 1.195
Joints:
- removed joint back_left_support_drone_to_payload
- removed joint back_right_support_drone_to_payload
- removed joint base_link_to_back_left_support_drone
- removed joint base_link_to_back_right_support_drone
- removed joint base_link_to_front_left_support_drone
- removed joint base_link_to_front_right_support_drone
- removed joint front_left_support_drone_to_payload
- removed joint front_right_support_drone_to_payload
