Commit message: 改变推力参数。明天细调

File: resources/robots/lmf2/model.urdf (robot description, URDF)
Before this commit: robot quadrotor, 5 links, 4 joints
Links:
- link base_link: mass 1.2 -> 12.0

Commit message: 一直会出现快速撞毁

File: resources/robots/lmf2/model.urdf (robot description, URDF)
Before this commit: robot quadrotor, 5 links, 4 joints
Links:
- link base_link: geometry collision box size=0.4 0.4 0.04; visual box size=0.4 0.4 0.025

Commit message: 修改Lmf2和控制器

File: resources/robots/lmf2/model.urdf (robot description, URDF)
Before this commit: robot quadrotor, 5 links, 4 joints
Links:
- added link payload_1_base, mass 1.0; visual box size=0.065 0.065 0.004; visual cylinder length=0.012 radius=0.008
- added link payload_2_base, mass 1.0; visual box size=0.065 0.065 0.004; visual cylinder length=0.012 radius=0.008
- added link payload_3_base, mass 1.0; visual box size=0.065 0.065 0.004; visual cylinder length=0.012 radius=0.008
- added link payload_4_base, mass 1.0; visual box size=0.065 0.065 0.004; visual cylinder length=0.012 radius=0.008
- link back_left_prop: geometry visual cylinder length=0.05 radius=0.015; visual cylinder length=0.18385 radius=0.01
- link back_right_prop: geometry visual cylinder length=0.05 radius=0.015; visual cylinder length=0.18385 radius=0.01
- link base_link: mass 12.0 -> 8.0; geometry collision box size=0.5 0.5 0.5; visual sphere radius=0.05
- link front_left_prop: geometry visual cylinder length=0.05 radius=0.015; visual cylinder length=0.18385 radius=0.01
- link front_right_prop: geometry visual cylinder length=0.05 radius=0.015; visual cylinder length=0.18385 radius=0.01
Joints:
- added joint base_link_to_payload_1: type fixed, parent base_link, child payload_1_base, origin xyz=0.0919 0.0919 -0.13
- added joint base_link_to_payload_2: type fixed, parent base_link, child payload_2_base, origin xyz=0.0919 -0.0919 -0.13
- added joint base_link_to_payload_3: type fixed, parent base_link, child payload_3_base, origin xyz=-0.0919 -0.0919 -0.13
- added joint base_link_to_payload_4: type fixed, parent base_link, child payload_4_base, origin xyz=-0.0919 0.0919 -0.13
- joint base_link_to_back_left_prop: origin xyz=-0.100 0.100 0 -> xyz=-0.13 0.13 0
- joint base_link_to_back_right_prop: origin xyz=-0.100 -0.100 0 -> xyz=-0.13 -0.13 0
- joint base_link_to_front_left_prop: origin xyz=0.100 0.100 0 -> xyz=0.13 0.13 0
- joint base_link_to_front_right_prop: origin xyz=0.100 -0.100 0 -> xyz=0.13 -0.13 0
