Commit message: 太久没有保存了 突然发现训练超参数和默认的有些不一样 以及大幅度加大方向奖励是没有作用的

File: resources/models/environment_assets/walls/back_wall.urdf (robot description, URDF)
Before this commit: robot back_wall, 1 links, 0 joints
Links:
- link base_link: geometry collision box size=0.2 50 40; visual box size=0.2 50 40

File: resources/models/environment_assets/walls/bottom_wall.urdf (robot description, URDF)
Before this commit: robot bottom_wall, 1 links, 0 joints
Links:
- link base_link: geometry collision box size=50 50 0.2; visual box size=50 50 0.2

File: resources/models/environment_assets/walls/front_wall.urdf (robot description, URDF)
Before this commit: robot front_wall, 1 links, 0 joints
Links:
- link base_link: geometry collision box size=0.2 50 40; visual box size=0.2 50 40

File: resources/models/environment_assets/walls/left_wall.urdf (robot description, URDF)
Before this commit: robot left_wall, 1 links, 0 joints
Links:
- link base_link: geometry collision box size=50 0.2 40; visual box size=50 0.2 40

File: resources/models/environment_assets/walls/right_wall.urdf (robot description, URDF)
Before this commit: robot right_wall, 1 links, 0 joints
Links:
- link base_link: geometry collision box size=50 0.2 40; visual box size=50 0.2 40

File: resources/models/environment_assets/walls/top_wall.urdf (robot description, URDF)
Before this commit: robot top_wall, 1 links, 0 joints
Links:
- link base_link: geometry collision box size=50 50 0.2; visual box size=50 50 0.2
